Commit message: Fixed maximal velocity of the simulated car

File: racer_description/urdf/racer_macros.xacro (robot description, xacro)
@@ -52,5 +52,5 @@
       <origin xyz="${translateX * OffsetJointX} ${translateY * OffsetJointY} ${OffsetJointZ}" rpy="0 0 0" />
       <axis xyz="0 1 0" rpy="0 0 0" />
-      <limit effort="10" velocity="100"/>
+      <limit effort="20" velocity="500"/>
       <joint_properties damping="0.0" friction="0.0"/>
     </joint>
