Commit message: Fix URDF conversion error

File: racer_description/urdf/racer.xacro (robot description, xacro)
@@ -1,4 +1,5 @@
 <?xml version='1.0'?>
-<robot name="myrobot" xmlns:xacro="http://www.ros.org/wiki/xacro">
+<robot name="myrobot"
+  xmlns:xacro="http://www.ros.org/wiki/xacro">
   <xacro:include filename="$(find racer_description)/urdf/racer_plugins.gazebo" />
   <xacro:include filename="$(find racer_description)/urdf/racer_macros.xacro" />
@@ -24,5 +25,5 @@
       <mass value="${bodyMass}"/>
       <origin xyz="0 0 ${wheel_height/2}" rpy=" 0 0 0"/>
-      <box_inertia  m="${bodyMass}" l="${bodySizeL}" b="${bodySizeB}" h="${bodySizeH}" />
+      <box_inertia m="${bodyMass}" l="${bodySizeL}" b="${bodySizeB}" h="${bodySizeH}" />
     </inertial>
     <collision name='collision'>
@@ -35,24 +36,16 @@
       <origin xyz="0 0 0" rpy=" 0 0 0"/>
       <geometry>
-         <mesh filename="package://racer_description/meshes/car.dae"/>
+        <mesh filename="package://racer_description/meshes/car.dae"/>
       </geometry>
     </visual>
   </link>
   <!--  Wheels  -->
-  <wheel fb="front" lr="left" parent="left_steering" translateX="1" translateY="1" left="1"
-  OffsetJointX= "${base_x_sphere_origin_to_wheel_origin}"  OffsetJointY= "${base_y_sphere_origin_to_wheel_origin}"
-  OffsetJointZ= "${base_z_sphere_origin_to_wheel_origin}" OffsetY="0.02" />
-  <wheel  fb="front" lr="right" parent="right_steering" translateX="1" translateY="-1" left="0"
-  OffsetJointX= "${base_x_sphere_origin_to_wheel_origin}"  OffsetJointY= "${base_y_sphere_origin_to_wheel_origin}"
-  OffsetJointZ= "${base_z_sphere_origin_to_wheel_origin}" OffsetY="-0.02" />
-  <wheel  fb="back" lr="left" parent="chassis" translateX="-1" translateY="1" left="1"
-  OffsetJointX= "${base_x_origin_to_wheel_origin}"  OffsetJointY= "${base_y_origin_to_wheel_origin}"
-  OffsetJointZ= "${base_z_origin_to_wheel_origin}" OffsetY="0.021" />
-  <wheel  fb="back" lr="right" parent="chassis" translateX="-1" translateY="-1" left="0"
-  OffsetJointX= "${base_x_origin_to_wheel_origin}"  OffsetJointY= "${base_y_origin_to_wheel_origin}"
-  OffsetJointZ= "${base_z_origin_to_wheel_origin}" OffsetY="-0.021" />
+  <wheel fb="front" lr="left" parent="left_steering" translateX="1" translateY="1" left="1" OffsetJointX= "${base_x_sphere_origin_to_wheel_origin}" OffsetJointY= "${base_y_sphere_origin_to_wheel_origin}" OffsetJointZ= "${base_z_sphere_origin_to_wheel_origin}" OffsetY="0.02" />
+  <wheel fb="front" lr="right" parent="right_steering" translateX="1" translateY="-1" left="0" OffsetJointX= "${base_x_sphere_origin_to_wheel_origin}" OffsetJointY= "${base_y_sphere_origin_to_wheel_origin}" OffsetJointZ= "${base_z_sphere_origin_to_wheel_origin}" OffsetY="-0.02" />
+  <wheel fb="back" lr="left" parent="chassis" translateX="-1" translateY="1" left="1" OffsetJointX= "${base_x_origin_to_wheel_origin}" OffsetJointY= "${base_y_origin_to_wheel_origin}" OffsetJointZ= "${base_z_origin_to_wheel_origin}" OffsetY="0.021" />
+  <wheel fb="back" lr="right" parent="chassis" translateX="-1" translateY="-1" left="0" OffsetJointX= "${base_x_origin_to_wheel_origin}" OffsetJointY= "${base_y_origin_to_wheel_origin}" OffsetJointZ= "${base_z_origin_to_wheel_origin}" OffsetY="-0.021" />
   <!-- Steering -->
-  <steering_hinge  lr="left" parent="chassis" translateY="1" OffsetY="0.01" />
-  <steering_hinge  lr="right" parent="chassis" translateY="-1" OffsetY="-0.01" />
+  <steering_hinge lr="left" parent="chassis" translateY="1" OffsetY="0.01" />
+  <steering_hinge lr="right" parent="chassis" translateY="-1" OffsetY="-0.01" />
   <!-- Camera -->
   <link name="camera">
@@ -71,5 +64,5 @@
       <origin xyz="0 0 0" rpy="0 0 0"/>
       <geometry>
-         <mesh filename="package://racer_description/meshes/ZED.dae"/>
+        <mesh filename="package://racer_description/meshes/ZED.dae"/>
       </geometry>
     </visual>
@@ -77,5 +70,5 @@
   <joint name="camera_joint" type="fixed">
     <axis xyz="0 1 0" />
-    <origin xyz=".21 0 0.075" rpy="0 0 0"/>
+    <origin xyz="0.21 0 0.075" rpy="0 0 0"/>
     <parent link="chassis"/>
     <child link="camera"/>
@@ -86,10 +79,10 @@
       <mass value="${hokuyoMass}" />
       <origin xyz="0 0 ${wheel_height/2}" rpy="0 0 0"/>
-      <box_inertia  m="${hokuyoMass}" l="${hokuyoSize}" b="${hokuyoSize}" h="${hokuyoSize}" />
+      <box_inertia m="${hokuyoMass}" l="${hokuyoSize}" b="${hokuyoSize}" h="${hokuyoSize}" />
     </inertial>
     <collision>
       <origin xyz="0 0 ${wheel_height/2}" rpy="0 0 0"/>
       <geometry>
-    	  <box size="${hokuyoSize} ${hokuyoSize} ${hokuyoSize}"/>
+        <box size="${hokuyoSize} ${hokuyoSize} ${hokuyoSize}"/>
       </geometry>
     </collision>
@@ -103,5 +96,5 @@
   <joint name="hokuyo_joint" type="fixed">
     <axis xyz="0 1 0" />
-    <origin xyz=".21 0 .135" rpy="0 0 0"/>
+    <origin xyz="0.21 0 0.135" rpy="0 0 0"/>
     <parent link="chassis"/>
     <child link="hokuyo"/>

Commit message: Add better IMU simulation

File: racer_description/urdf/racer.xacro (robot description, xacro)
@@ -10,4 +10,6 @@
   <xacro:property name="hokuyoSize" value="0.1"/>
   <xacro:property name="hokuyoMass" value="0.1"/>
+  <xacro:property name="imuSize" value="0.1"/>
+  <xacro:property name="imuMass" value="0.1"/>
   <xacro:property name="bodySizeL" value="0.49"/>
   <xacro:property name="bodySizeB" value="0.18"/>
@@ -100,3 +102,29 @@
     <child link="laser"/>
   </joint>
+  <!-- IMU -->
+  <link name="imu_link">
+    <inertial>
+      <mass value="${imuMass}" />
+      <origin xyz="0 0 ${wheel_height/2}" rpy="0 0 0"/>
+      <box_inertia m="${imuMass}" l="${imuSize}" b="${imuSize}" h="${imuSize}" />
+    </inertial>
+    <collision>
+      <origin xyz="0 0 ${wheel_height/2}" rpy="0 0 0"/>
+      <geometry>
+        <box size="${imuSize} ${imuSize} ${imuSize}"/>
+      </geometry>
+    </collision>
+    <visual>
+      <origin xyz="0 0 ${wheel_height/2}" rpy="0 0 0"/>
+      <geometry>
+        <box size="${imuSize} ${imuSize} ${imuSize}"/>
+      </geometry>
+    </visual>
+  </link>
+  <joint name="imu_joint" type="fixed">
+    <axis xyz="0 1 0" />
+    <origin xyz="0 0 0.135" rpy="0 0 0"/>
+    <parent link="chassis"/>
+    <child link="imu_link"/>
+  </joint>
 </robot>

Commit message: Update the name of the laser scanner frame in some more places

File: racer_description/urdf/racer.xacro (robot description, xacro)
@@ -75,5 +75,5 @@
   </joint>
   <!-- Hokuyo Laser -->
-  <link name="hokuyo">
+  <link name="laser">
     <inertial>
       <mass value="${hokuyoMass}" />
@@ -94,9 +94,9 @@
     </visual>
   </link>
-  <joint name="hokuyo_joint" type="fixed">
+  <joint name="laser_joint" type="fixed">
     <axis xyz="0 1 0" />
     <origin xyz="0.21 0 0.135" rpy="0 0 0"/>
     <parent link="chassis"/>
-    <child link="hokuyo"/>
+    <child link="laser"/>
   </joint>
 </robot>

Commit message: Remove IMU inertial, collision, visual

File: racer_description/urdf/racer.xacro (robot description, xacro)
@@ -103,23 +103,5 @@
   </joint>
   <!-- IMU -->
-  <link name="imu_link">
-    <inertial>
-      <mass value="${imuMass}" />
-      <origin xyz="0 0 ${wheel_height/2}" rpy="0 0 0"/>
-      <box_inertia m="${imuMass}" l="${imuSize}" b="${imuSize}" h="${imuSize}" />
-    </inertial>
-    <collision>
-      <origin xyz="0 0 ${wheel_height/2}" rpy="0 0 0"/>
-      <geometry>
-        <box size="${imuSize} ${imuSize} ${imuSize}"/>
-      </geometry>
-    </collision>
-    <visual>
-      <origin xyz="0 0 ${wheel_height/2}" rpy="0 0 0"/>
-      <geometry>
-        <box size="${imuSize} ${imuSize} ${imuSize}"/>
-      </geometry>
-    </visual>
-  </link>
+  <link name="imu_link" />
   <joint name="imu_joint" type="fixed">
     <axis xyz="0 1 0" />

Commit message: Remove imuSize & imuMass

File: racer_description/urdf/racer.xacro (robot description, xacro)
@@ -10,6 +10,4 @@
   <xacro:property name="hokuyoSize" value="0.1"/>
   <xacro:property name="hokuyoMass" value="0.1"/>
-  <xacro:property name="imuSize" value="0.1"/>
-  <xacro:property name="imuMass" value="0.1"/>
   <xacro:property name="bodySizeL" value="0.49"/>
   <xacro:property name="bodySizeB" value="0.18"/>

Commit message: Added car highlighting

File: racer_description/urdf/racer.xacro (robot description, xacro)
@@ -14,4 +14,5 @@
   <xacro:property name="bodySizeH" value="0.1"/>
   <xacro:property name="bodyMass" value="3.5"/>
+  <xacro:arg name="car_highlighting" default="false"/>
   <link name="base_link" />
   <joint name="base_link_joint" type="fixed">
@@ -40,4 +41,9 @@
     </visual>
   </link>
+  <xacro:if value="$(arg car_highlighting)">
+    <gazebo reference="chassis">
+      <material>Gazebo/GreenGlow</material>
+    </gazebo>
+  </xacro:if>
   <!--  Wheels  -->
   <wheel fb="front" lr="left" parent="left_steering" translateX="1" translateY="1" left="1" OffsetJointX= "${base_x_sphere_origin_to_wheel_origin}" OffsetJointY= "${base_y_sphere_origin_to_wheel_origin}" OffsetJointZ= "${base_z_sphere_origin_to_wheel_origin}" OffsetY="0.02" />

Commit message: Add car body

File: racer_description/urdf/racer.xacro (robot description, xacro)
@@ -38,4 +38,17 @@
       <geometry>
         <mesh filename="package://racer_description/meshes/car.dae"/>
+      </geometry>
+    </visual>
+  </link>
+  <joint name="base_body_joint" type="fixed">
+    <origin xyz="0 0 0" rpy="0 0 0" />
+    <parent link="base_link" />
+    <child link="body" />
+  </joint>
+  <link name='body'>
+    <visual>
+      <origin xyz="0 0 0.05" rpy=" 0 0 0"/>
+      <geometry>
+        <mesh filename="package://racer_description/meshes/body.dae"/>
       </geometry>
     </visual>

Commit message: Update the positon of the camera

File: racer_description/urdf/racer.xacro (robot description, xacro)
@@ -89,5 +89,5 @@
   <joint name="camera_joint" type="fixed">
     <axis xyz="0 1 0" />
-    <origin xyz="0.21 0 0.075" rpy="0 0 0"/>
+    <origin xyz="0.21 0 0.095" rpy="0 0 0"/>
     <parent link="chassis"/>
     <child link="camera"/>

Commit message: Remove car highlighting since the car is always brightly visible

File: racer_description/urdf/racer.xacro (robot description, xacro)
@@ -14,5 +14,4 @@
   <xacro:property name="bodySizeH" value="0.1"/>
   <xacro:property name="bodyMass" value="3.5"/>
-  <xacro:arg name="car_highlighting" default="false"/>
   <link name="base_link" />
   <joint name="base_link_joint" type="fixed">
@@ -54,9 +53,4 @@
     </visual>
   </link>
-  <xacro:if value="$(arg car_highlighting)">
-    <gazebo reference="chassis">
-      <material>Gazebo/GreenGlow</material>
-    </gazebo>
-  </xacro:if>
   <!--  Wheels  -->
   <wheel fb="front" lr="left" parent="left_steering" translateX="1" translateY="1" left="1" OffsetJointX= "${base_x_sphere_origin_to_wheel_origin}" OffsetJointY= "${base_y_sphere_origin_to_wheel_origin}" OffsetJointZ= "${base_z_sphere_origin_to_wheel_origin}" OffsetY="0.02" />
